File: board.kicad_sch (KiCad schematic)
At the start: 34 parts, among them J1 Conn_02x16_Odd_Even, J2 JSTBATT, Q1 2N7002, SW1 SW_SPDT, U1 BQ24075RGT, U2 nRF52840_holyiot_18010, U3 XC6206PxxxMR, U4 SRV05-4

Commit message: Updated to revision 0.2, with Holyiot module on edge of board
Connections:
- net +BATT: now also R10.1
- net +VSW: no longer R10.1
- net P0.06: now also J1.25 (Pin_25); no longer J1.26 (Pin_26)
- net P0.08: now also J1.24 (Pin_24); no longer J1.23 (Pin_23)
- net P0.11: now also J1.21 (Pin_21); no longer J1.22 (Pin_22)
- net P0.25: now also J1.20 (Pin_20); no longer J1.19 (Pin_19)
- net P0.26: now also J1.26 (Pin_26); no longer J1.25 (Pin_25)
- net P0.27: now also J1.23 (Pin_23); no longer J1.24 (Pin_24)
- net P1.08: now also J1.22 (Pin_22); no longer J1.21 (Pin_21)
- net P1.12: now also J1.19 (Pin_19); no longer J1.20 (Pin_20)
Changed lines of the file:
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@@
 	(title_block
 		(title "nRF52840-Uno")
-		(date "2024-08-12")
-		(rev "0.1")
+		(date "2024-08-13")
+		(rev "0.2")
 		(company "Scott O'Brien")
 	)
@@
 	)
 	(label "P0.26"
-		(at 133.35 124.46 180)
+		(at 146.05 124.46 0)
 		(fields_autoplaced yes)
 		(effects
@@
 				(size 1.27 1.27)
 			)
-			(justify right bottom)
+			(justify left bottom)
 		)
 	)
@@
 	)
 	(label "P0.27"
-		(at 146.05 121.92 0)
+		(at 133.35 121.92 180)
 		(fields_autoplaced yes)
 		(effects
@@
 				(size 1.27 1.27)
 			)
-			(justify left bottom)
+			(justify right bottom)
 		)
 	)
@@
 	)
 	(label "P1.12"
-		(at 146.05 116.84 0)
+		(at 133.35 116.84 180)
 		(fields_autoplaced yes)
 		(effects
@@
 				(size 1.27 1.27)
 			)
-			(justify left bottom)
+			(justify right bottom)
 		)
 	)
@@
 	)
 	(label "P0.25"
-		(at 133.35 116.84 180)
+		(at 146.05 116.84 0)
 		(fields_autoplaced yes)
 		(effects
@@
 				(size 1.27 1.27)
 			)
-			(justify right bottom)
+			(justify left bottom)
 		)
 	)
@@
 	)
 	(label "P0.11"
-		(at 146.05 119.38 0)
+		(at 133.35 119.38 180)
 		(fields_autoplaced yes)
 		(effects
@@
 				(size 1.27 1.27)
 			)
-			(justify left bottom)
+			(justify right bottom)
 		)
 	)
@@
 	)
 	(label "P0.06"
-		(at 146.05 124.46 0)
+		(at 133.35 124.46 180)
 		(fields_autoplaced yes)
 		(effects
@@
 				(size 1.27 1.27)
 			)
-			(justify left bottom)
+			(justify right bottom)
 		)
 	)
@@
 	)
 	(label "P0.08"
-		(at 133.35 121.92 180)
+		(at 146.05 121.92 0)
 		(fields_autoplaced yes)
 		(effects
@@
 				(size 1.27 1.27)
 			)
-			(justify right bottom)
+			(justify left bottom)
 		)
 	)
@@
 	)
 	(label "P1.08"
-		(at 133.35 119.38 180)
+		(at 146.05 119.38 0)
 		(fields_autoplaced yes)
 		(effects
@@
 				(size 1.27 1.27)
 			)
-			(justify right bottom)
+			(justify left bottom)
 		)
 	)
@@
 	)
 	(symbol
-		(lib_id "power:+VSW")
-		(at 231.14 134.62 0)
-		(unit 1)
-		(exclude_from_sim no)
-		(in_bom yes)
-		(on_board yes)
-		(dnp no)
-		(fields_autoplaced yes)
-		(property "Reference" "#PWR026"
-			(at 231.14 138.43 0)
-			(effects
-				(font
-					(size 1.27 1.27)
-				)
-				(hide yes)
-			)
-		)
-		(property "Value" "+VSW"
-			(at 231.14 129.54 0)
-			(effects
-				(font
-					(size 1.27 1.27)
-				)
-			)
-		)
-		(property "Footprint" ""
-			(at 231.14 134.62 0)
-			(effects
-				(font
-					(size 1.27 1.27)
-				)
-				(hide yes)
-			)
-		)
-		(property "Datasheet" ""
-			(at 231.14 134.62 0)
-			(effects
-				(font
-					(size 1.27 1.27)
-				)
-				(hide yes)
-			)
-		)
-		(property "Description" "Power symbol creates a global label with name \"+VSW\""
-			(at 231.14 134.62 0)
-			(effects
-				(font
-					(size 1.27 1.27)
-				)
-				(hide yes)
-			)
-		)
-		(pin "1"
-		)
-		(instances
-			(project "board"
-				(path "/1e24de4f-8603-46cc-9c9d-c795d003639a"
-					(reference "#PWR026")
-					(unit 1)
-				)
-			)
-		)
-	)
-	(symbol
 		(lib_id "Device:R")
 		(at 231.14 146.05 0)
@@
 					(unit 1)
 				)
+			)
+		)
+	)
+	(symbol
+		(lib_id "power:+BATT")
+		(at 231.14 134.62 0)
+		(unit 1)
+		(exclude_from_sim no)
+		(in_bom yes)
+		(on_board yes)
+		(dnp no)
+		(fields_autoplaced yes)
+		(property "Reference" "#PWR026"
+			(at 231.14 138.43 0)
+			(effects
+				(font
+					(size 1.27 1.27)
+				)
+				(hide yes)
+			)
+		)
+		(property "Value" "+BATT"
+			(at 231.14 129.54 0)
+			(effects
+				(font
+					(size 1.27 1.27)
+				)
+			)
+		)
+		(property "Footprint" ""
+			(at 231.14 134.62 0)
+			(effects
+				(font
+					(size 1.27 1.27)
+				)
+				(hide yes)
+			)
+		)
+		(property "Datasheet" ""
+			(at 231.14 134.62 0)
+			(effects
+				(font
+					(size 1.27 1.27)
+				)
+				(hide yes)
+			)
+		)
+		(property "Description" "Power symbol creates a global label with name \"+BATT\""
+			(at 231.14 134.62 0)
+			(effects
+				(font
+					(size 1.27 1.27)
+				)
+				(hide yes)
+			)
+		)
+		(pin "1"
+		)
+		(instances
+			(project "board"
+				(path "/1e24de4f-8603-46cc-9c9d-c795d003639a"
+					(reference "#PWR026")
+					(unit 1)
+				)

Commit message: Added debug / programming pins
Parts:
- added J3: Conn_01x02_Socket, Connector_PinHeader_2.54mm:PinHeader_1x02_P2.54mm_Vertical, symbol Connector:Conn_01x02_Socket
- C1: footprint LED_SMD:LED_0402_1005Metric -> Capacitor_SMD:C_0603_1608Metric
- F1: footprint Fuse:Fuse_0402_1005Metric -> Fuse:Fuse_0805_2012Metric
- LED_CHG1: footprint LED_SMD:LED_0402_1005Metric -> LED_SMD:LED_0603_1608Metric_Pad1.05x0.95mm_HandSolder
- R1, R10, R11, R12, R13, R2, R3, R4, R5, R6, R7, R8, R9: footprint Resistor_SMD:R_0402_1005Metric -> Resistor_SMD:R_0603_1608Metric_Pad0.98x0.95mm_HandSolder
- R14: footprint Resistor_SMD:R_0603_1608Metric -> Resistor_SMD:R_0603_1608Metric_Pad0.98x0.95mm_HandSolder
Connections:
- net +3.3V: now also J3.2 (Pin_2)
- net +BATT: no longer R10.1
- net +VSW: now also R10.1
- net GND: now also J3.1 (Pin_1)
Other:
- note added: "Debug Pins"

Commit message: Fixed polarity of connector
Connections:
- net +BATT: now also J2.2 (Pin_2); no longer J2.1 (Pin_1)
- net GND: now also J2.1 (Pin_1); no longer J2.2 (Pin_2)
